File: Clap-pixel-board/Clap-pixel-board.kicad_pcb (KiCad board)
At the start: 4 copper layers, 100 x 70 mm, 41 parts, among them J1 USB_C_6P, J2 ST-Link, J3 TC2030-NL, U1 AP2210N-3.3TRG1, U2 STM32G070CBTx, U3 74AHCT1G125SE-7

Commit message: Finished PCB
Parts:
- moved C13 3.97 mm to (168.2, 79.5)
- moved C11 3.55 mm to (151.8, 120.4)
- moved C10 3.55 mm to (128.2, 119.5), turned to 90 degrees
- moved C14 3.55 mm to (168.2, 119.6), turned to 90 degrees
- moved C12 0.73 mm to (151.8, 80.5), turned to -90 degrees
- moved C15 0.34 mm to (138.1, 85.5)
- moved C4 0.20 mm to (177.2, 99.8)
- moved C9 0.11 mm to (128.2, 79.5)
- turned D3 to -90 degrees
- turned D4 to -90 degrees
Routing:
- net /DIN2: track 0.00 -> 42.4 mm, vias 0 -> 2
- net /DIN6: track 0.00 -> 41.6 mm
- net /DIN4: track 0.00 -> 38.6 mm, vias 0 -> 2
- net VBUS: track 0.00 -> 30.6 mm, vias 0 -> 10
- net NRST: track 0.00 -> 26.9 mm, vias 0 -> 2
- net SWDIO: track 0.00 -> 23.1 mm
- net /DIN3: track 0.00 -> 22.5 mm
- net /DIN5: track 0.00 -> 22.0 mm
- net RX: track 0.00 -> 20.5 mm
- net SWCLK: track 0.00 -> 18.8 mm, vias 0 -> 2
- net +3V3: track 0.00 -> 16.1 mm, vias 0 -> 12
- net MIC: track 0.00 -> 15.5 mm
- net TX: track 0.00 -> 14.9 mm
- net /DIN1: track 0.00 -> 14.7 mm
- net NEO_IN: track 0.00 -> 9.41 mm
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- added copper zone on In2.Cu, net +3V3
- added copper zone on B.Cu, net GND
- added copper zone on F.Cu, net GND
- added copper zone on In1.Cu, net GND
- added copper zone on In2.Cu, net VBUS
